File: ft2232-breakout.kicad_sch (KiCad schematic)
At the start: 59 parts, among them J1 USB_C_Receptacle_USB2.0, J2 Conn_01x20, J3 Conn_01x20, J4 Conn_01x07, J5 Conn_01x07, J6 Conn_01x06, J7 Conn_01x06, U2 MIC5205-3.3YM5, U3 FT2232HL, U4 93LC46BT-I/OT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

Commit message: Oct2022 as manufactured
Parts:
- C25: value NF -> 100n
- R11: value 330 -> 1k
- R4: value 330 -> 1k; symbol Device:R -> Device:R_Small
Changed lines of the file:
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@@
     (stroke (width 0) (type default) (color 0 0 0 0))
   )
-  (wire (pts (xy 180.34 22.86) (xy 180.34 24.13))
+  (wire (pts (xy 180.34 22.86) (xy 180.34 25.4))
     (stroke (width 0) (type default) (color 0 0 0 0))
   )
-  (wire (pts (xy 180.34 34.29) (xy 180.34 31.75))
+  (wire (pts (xy 180.34 30.48) (xy 180.34 34.29))
     (stroke (width 0) (type default) (color 0 0 0 0))
   )
@@
     (stroke (width 0) (type default) (color 0 0 0 0))
   )
-  (wire (pts (xy 33.02 71.12) (xy 33.02 69.85))
+  (wire (pts (xy 33.02 78.105) (xy 33.02 69.85))
     (stroke (width 0) (type default) (color 0 0 0 0))
   )
@@
     (pin "1")
   )
-  (symbol (lib_id "power:GND") (at 33.02 71.12 0) (unit 1)
+  (symbol (lib_id "power:GND") (at 33.02 78.105 0) (unit 1)
     (in_bom yes) (on_board yes)
-    (property "Reference" "#PWR0103" (id 0) (at 33.02 77.47 0)
+    (property "Reference" "#PWR0103" (id 0) (at 33.02 84.455 0)
       (effects (font (size 1.27 1.27)) hide)
     )
-    (property "Value" "GND" (id 1) (at 33.147 75.5142 0))
-    (property "Footprint" "" (id 2) (at 33.02 71.12 0)
+    (property "Value" "GND" (id 1) (at 33.147 82.4992 0))
+    (property "Footprint" "" (id 2) (at 33.02 78.105 0)
       (effects (font (size 1.27 1.27)) hide)
     )
-    (property "Datasheet" "" (id 3) (at 33.02 71.12 0)
+    (property "Datasheet" "" (id 3) (at 33.02 78.105 0)
       (effects (font (size 1.27 1.27)) hide)
     )
@@
     (pin "1")
   )
-  (symbol (lib_id "Device:R") (at 180.34 27.94 0) (unit 1)
+  (symbol (lib_id "Device:R_Small") (at 180.34 27.94 0) (unit 1)
     (in_bom yes) (on_board yes)
     (property "Reference" "R4" (id 0) (at 182.118 26.7716 0)
       (effects (font (size 1.27 1.27)) (justify left))
     )
-    (property "Value" "330" (id 1) (at 182.118 29.083 0)
+    (property "Value" "1k" (id 1) (at 182.118 29.083 0)
       (effects (font (size 1.27 1.27)) (justify left))
     )
-    (property "Footprint" "Inductor_SMD:L_0805_2012Metric" (id 2) (at 178.562 27.94 90)
+    (property "Footprint" "Inductor_SMD:L_0805_2012Metric" (id 2) (at 180.34 27.94 0)
       (effects (font (size 1.27 1.27)) hide)
     )
@@
     (in_bom yes) (on_board yes)
     (property "Reference" "C25" (id 0) (at 29.21 73.3298 90))
-    (property "Value" "NF" (id 1) (at 29.21 75.6412 90))
+    (property "Value" "100n" (id 1) (at 29.21 75.6412 90))
     (property "Footprint" "Capacitor_SMD:C_0805_2012Metric" (id 2) (at 29.21 69.85 0)
       (effects (font (size 1.27 1.27)) hide)
@@
       (effects (font (size 1.27 1.27)) (justify right))
     )
-    (property "Value" "330" (id 1) (at 148.1836 197.993 0)
+    (property "Value" "1k" (id 1) (at 148.1836 197.993 0)
       (effects (font (size 1.27 1.27)) (justify right))
     )
@@
     )
     (path "/00000000-0000-0000-0000-00005f3a982f"
-      (reference "C25") (unit 1) (value "NF") (footprint "Capacitor_SMD:C_0805_2012Metric")
+      (reference "C25") (unit 1) (value "100n") (footprint "Capacitor_SMD:C_0805_2012Metric")
     )
     (path "/00000000-0000-0000-0000-00005fa89fd4"
@@
     )
     (path "/00000000-0000-0000-0000-00005ec7911b"
-      (reference "R4") (unit 1) (value "330") (footprint "Inductor_SMD:L_0805_2012Metric")
+      (reference "R4") (unit 1) (value "1k") (footprint "Inductor_SMD:L_0805_2012Metric")
     )
     (path "/00000000-0000-0000-0000-00005ee10d01"
@@
     )
     (path "/00000000-0000-0000-0000-000060280318"
-      (reference "R11") (unit 1) (value "330") (footprint "Inductor_SMD:L_0805_2012Metric")
+      (reference "R11") (unit 1) (value "1k") (footprint "Inductor_SMD:L_0805_2012Metric")
     )
     (path "/00000000-0000-0000-0000-00005f33b0f5"
